File: projects/boiler_themp/PLM_1/modem_tda.sch (EAGLE design)
At the start: 17 parts, among them IC1 TDA5051, X1 8MHz

Commit message: PLM Version 1.0 Finished and sent to PCB house
Parts:
- added C3: 10 uF 16V, ipc-7351-capacitor:CAPACITOR_1206
- added C4: 100 uF, ipc-7351-capacitor:POLARISED_U_CASE
- added C5: 0.1uF, ipc-7351-capacitor:CAPACITOR_0805
- added D1: SMBJ7.0A, diode:SUPPRESSOR-SMBJ
- added JP1: (no value), jlab:BLUE_TERM
- added L1: 47 uH, jlab_varistors:L-US
- added L2: 22 uH, jlab_varistors:L-US
- added OC1: PC814, optocoupler:PC814
- added Q1: 2N3904SOT23, transistor-npn:2N3904SOT23
- added R6: 10D391K, jlab_varistors:VARISTOR
- added SV1: (no value), con-lstb:MA06-1
- added T1: MU-78250, jlab:MU-78250
- F1: device fuse:FUSESHK20L -> fuse:SHK20L
- R2: device rcl:R-EU_0207/10 -> rcl:R-EU_0309/12
Connections:
- new net +5V: C4.+, C7.2, C8.2, IC1.VDDA, IC1.VDDAP, IC1.VDDD, OC1.C, R5.2, SV1.1
- new net GND: C1.2, C10.1, C2.2, C4.-, C5.1, C7.1, C8.1, D1.A, IC1.AGND, IC1.APGND, IC1.DGND, L2.1, Q1.E, R1.1, R8.1, SV1.5, SV1.6, T1.1
- new net N$1: F1.1A, F1.1B, JP1.2
- new net N$10: C10.2, Q1.C, R5.1, SV1.2
- new net N$11: C6.1, IC1.RXIN
- new net N$12: C2.1, IC1.OSC1, R7.2, X1.2
- new net N$13: C1.1, IC1.OSC2, R7.1, X1.1
- new net N$14: IC1.DATAIN, SV1.3
- new net N$15: IC1.DATAOUT, SV1.4
- new net N$16: Q1.B, R4.2
- new net N$2: F1.2A, F1.2B, R2.1, R3.2, R6.2, T1.4
- new net N$3: C9.1, JP1.1, OC1.AC1, R3.1, R6.1
- new net N$4: OC1.AC2, R2.2
- new net N$5: C9.2, L1.2
- new net N$6: L1.1, T1.6
- new net N$7: OC1.E, R4.1, R8.2
- new net N$8: C3.1, C5.2, L2.2, R1.2, T1.3
- new net N$9: C3.2, C6.2, D1.C, IC1.TXOUT
Other:
- moved on the sheet: C1, C10, C2, C6, C7, C8, C9, IC1, R1, R2, R3, R4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
