File: projects/STM32/STM32F103_my_launchpad/stm32f103_pin1.brd (EAGLE design)
At the start: 50 x 50 mm, 52 parts, among them J1 USBMOLEX, Q1 8MHz, Q2 32768, U1 TLV1117, U2 STM32F103C8LQFP48

Commit message: stm32 launchpad ver 1.1
Parts:
- S1, S2: value DTE6 -> DT5X6; device jlab:DTE6 -> jlab:TACTILE-PTH
- U2: value STM32F103C8LQFP48 -> STM32F103C8MANUAL_SOLDER; device STM32_dhalt:LQFP48 -> STM32_dhalt:LQFP48_IGORL
- moved S2 0.76 mm to (4.57, 3.81)
- moved S1 0.63 mm to (45.1, 3.81)
- turned U2 to 0 degrees
Connections:
- net N$16: now also S2.4; no longer S2.3
- net N$5: now also S1.4; no longer S1.3
Routing:
- net N$16: track 5.08 -> 3.72 mm
- net N$5: track 22.9 -> 21.6 mm
- net N$20: track 8.80 -> 8.06 mm
- net +3V3: track 132.5 -> 131.9 mm
Other:
- board text added: "May 2013"
- board text added: "STM32F10xCxT6 base ver 1.1"
- board text removed: "Mar 2013"
- board text removed: "STM32F10xCxT6 base ver 1.0"
