File: projects/STM32/STM32F103_my_launchpad/stm32f103_pin1.sch (EAGLE design)
At the start: 52 parts, among them J1 USBMOLEX, Q1 8MHz, Q2 32768, U1 TLV1117, U2 STM32F103C8LQFP48

Commit message: stm32 launchpad ver 1.1
Parts:
- S1, S2: value DTE6 -> DT5X6; device jlab:DTE6 -> jlab:DT5X6
- U2: value STM32F103C8LQFP48 -> STM32F103C8MANUAL_SOLDER; device STM32_dhalt:STM32F103C8LQFP48 -> STM32_dhalt:STM32F103C8MANUAL_SOLDER
Changed lines of the file:
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@@
 <part name="R7" library="ipc-7351-resistor" deviceset="RESISTOR_" device="0805" value="680"/>
 <part name="R8" library="ipc-7351-resistor" deviceset="RESISTOR_" device="0805" value="510"/>
-<part name="S1" library="jlab" deviceset="DT" device="E6"/>
+<part name="S1" library="jlab" deviceset="DT" device="5X6"/>
 <part name="BOOT0" library="pinhead" deviceset="PINHD-1X3" device=""/>
 <part name="BOOT1" library="pinhead" deviceset="PINHD-1X3" device=""/>
@@
 <part name="GND7" library="supply1" deviceset="GND" device=""/>
 <part name="GND8" library="supply1" deviceset="GND" device=""/>
-<part name="S2" library="jlab" deviceset="DT" device="E6"/>
+<part name="S2" library="jlab" deviceset="DT" device="5X6"/>
 <part name="+3V2" library="supply1" deviceset="+3V3" device=""/>
 <part name="GND9" library="supply1" deviceset="GND" device=""/>
@@
 <part name="R12" library="ipc-7351-resistor" deviceset="RESISTOR_" device="0805" value="470"/>
 <part name="+3V11" library="supply1" deviceset="+3V3" device=""/>
-<part name="U2" library="STM32_dhalt" deviceset="STM32F103C8" device="LQFP48"/>
+<part name="U2" library="STM32_dhalt" deviceset="STM32F103C8" device="MANUAL_SOLDER" value="STM32F103C8MANUAL_SOLDER"/>
 <part name="+3V12" library="supply1" deviceset="+3V3" device=""/>
 <part name="+3V13" library="supply1" deviceset="+3V3" device=""/>
