File: projects/jphy.v1.3/jphy_v1.3.brd (EAGLE design)
At the start: 49 x 24 mm, 11 parts, among them IC1 MAX3232ESE, J1 RJ45-8X

Commit message: JPHY ver 1.3 (300 pcs)
Parts:
- C1, C2, C3, C4, C5: device rcl:C0805 -> ipc-7351-capacitor:CAPC2012X145AN
- R1: device rcl:R0805 -> ipc-7351-resistor:RESC2012X70N
Other:
- board text added: "Designed by Igor L."
- board text added: "JSERIAL v1.3"
- board text added: "Sep 2013"
- board text removed: "Igor L."
- board text removed: "JSERIAL v1.2"
- board text removed: "Nov 2012"
Changed lines of the file:
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@@
 <?xml version="1.0" encoding="utf-8"?>
 <!DOCTYPE eagle SYSTEM "eagle.dtd">
-<eagle version="6.3">
+<eagle version="6.5.0">
 <drawing>
 <settings>
@@
 <layer number="37" name="tTest" color="7" fill="1" visible="no" active="yes"/>
 <layer number="38" name="bTest" color="7" fill="1" visible="no" active="yes"/>
-<layer number="39" name="tKeepout" color="4" fill="11" visible="no" active="yes"/>
-<layer number="40" name="bKeepout" color="1" fill="11" visible="no" active="yes"/>
+<layer number="39" name="tKeepout" color="4" fill="11" visible="yes" active="yes"/>
+<layer number="40" name="bKeepout" color="1" fill="11" visible="yes" active="yes"/>
 <layer number="41" name="tRestrict" color="4" fill="10" visible="no" active="yes"/>
 <layer number="42" name="bRestrict" color="1" fill="10" visible="no" active="yes"/>
@@
 <layer number="48" name="Document" color="7" fill="1" visible="no" active="yes"/>
 <layer number="49" name="Reference" color="7" fill="1" visible="no" active="yes"/>
+<layer number="50" name="dxf" color="7" fill="1" visible="no" active="yes"/>
 <layer number="51" name="tDocu" color="7" fill="1" visible="yes" active="yes"/>
 <layer number="52" name="bDocu" color="7" fill="1" visible="yes" active="yes"/>
@@
 <layer number="97" name="Info" color="7" fill="1" visible="no" active="no"/>
 <layer number="98" name="Guide" color="6" fill="1" visible="no" active="no"/>
+<layer number="250" name="Descript" color="3" fill="1" visible="no" active="no"/>
+<layer number="251" name="SMDround" color="12" fill="11" visible="no" active="no"/>
 </layers>
 <board>
@@
 <circle x="9.525" y="13.335" radius="0.508" width="0" layer="25"/>
 <text x="27.94" y="10.16" size="0.8128" layer="25" font="vector" ratio="16" rot="R90">Vcc Rx Tx Gnd</text>
-<text x="22.86" y="21.59" size="1.778" layer="25">Nov 2012</text>
-<text x="22.86" y="12.7" size="1.4224" layer="26" font="vector" ratio="16" rot="MR0">JSERIAL v1.2</text>
-<text x="7.62" y="1.27" size="1.4224" layer="25" font="vector" ratio="13">Igor L.</text>
+<text x="22.86" y="21.59" size="1.778" layer="25">Sep 2013</text>
+<text x="22.86" y="12.7" size="1.4224" layer="26" font="vector" ratio="16" rot="MR0">JSERIAL v1.3</text>
+<text x="7.62" y="1.27" size="1.4224" layer="25" font="vector" ratio="13">Designed by Igor L.</text>
 <hole x="45.72" y="21.59" drill="3"/>
 </plain>
@@
 <attribute name="OC_NEWARK" value="79C3880" x="15.24" y="16.51" size="1.778" layer="27" display="off"/>
 </element>
-<element name="C1" library="rcl" package="C0805" value="0.47 uF" x="7.62" y="5.715" rot="R90"/>
-<element name="C2" library="rcl" package="C0805" value="0.47 uF" x="11.43" y="5.715" rot="R90"/>
-<element name="C3" library="rcl" package="C0805" value="0.47 uF" x="15.24" y="5.715" rot="R90"/>
-<element name="C4" library="rcl" package="C0805" value="0.47 uF" x="19.05" y="5.715" rot="R90"/>
-<element name="C5" library="rcl" package="C0805" value="0.47 uF" x="6.858" y="20.32" rot="R90"/>
-<element name="R1" library="rcl" package="R0805" value="270 R" x="24.13" y="5.715" rot="R90"/>
+<element name="C1" library="ipc-7351-capacitor" package="CAPC2012X145AN" value="0.47 uF" x="7.62" y="5.715" rot="R90"/>
+<element name="C2" library="ipc-7351-capacitor" package="CAPC2012X145AN" value="0.47 uF" x="11.43" y="5.715" rot="R90"/>
+<element name="C3" library="ipc-7351-capacitor" package="CAPC2012X145AN" value="0.47 uF" x="15.24" y="5.715" rot="R90"/>
+<element name="C4" library="ipc-7351-capacitor" package="CAPC2012X145AN" value="0.47 uF" x="19.05" y="5.715" rot="R90"/>
+<element name="C5" library="ipc-7351-capacitor" package="CAPC2012X145AN" value="0.47 uF" x="6.858" y="20.32" rot="R90"/>
+<element name="R1" library="ipc-7351-resistor" package="RESC2012X70N" value="270 R" x="24.13" y="5.715" rot="R90"/>
 <element name="LED1" library="jlab" package="CHIP-LED0805" value="Green" x="24.13" y="12.7" smashed="yes" rot="R180">
 <attribute name="NAME" x="20.701" y="14.605" size="1.27" layer="25" ratio="10" rot="R270"/>
@@
 </polygon>
 <via x="21.59" y="4.765" extent="1-16" drill="0.7" diameter="0.254"/>
-<wire x1="19.05" y1="4.765" x2="19.116" y2="4.699" width="0.8128" layer="1"/>
-<wire x1="21.59" y1="4.765" x2="19.05" y2="4.765" width="0.8128" layer="1"/>
+<wire x1="19.05" y1="4.815" x2="19.116" y2="4.699" width="0.8128" layer="1"/>
+<wire x1="21.59" y1="4.765" x2="19.05" y2="4.815" width="0.8128" layer="1"/>
 <wire x1="21.59" y1="4.765" x2="24.13" y2="4.765" width="0.8128" layer="1"/>
 <wire x1="8.763" y1="22.098" x2="7.935" y2="21.27" width="0.8128" layer="1"/>
-<wire x1="7.935" y1="21.27" x2="6.858" y2="21.27" width="0.8128" layer="1"/>
+<wire x1="7.935" y1="21.27" x2="6.858" y2="21.22" width="0.8128" layer="1"/>
 <via x="40.386" y="12.7" extent="1-16" drill="0.7"/>
 <polygon width="0.8128" layer="1">
@@
 <wire x1="41.91" y1="6.35" x2="41.91" y2="10.16" width="0.8128" layer="1"/>
 <wire x1="38.1" y1="2.54" x2="41.91" y2="6.35" width="0.8128" layer="1"/>
-<wire x1="15.24" y1="4.765" x2="15.24" y2="3.81" width="0.8128" layer="1"/>
+<wire x1="15.24" y1="4.815" x2="15.24" y2="3.81" width="0.8128" layer="1"/>
 <wire x1="15.24" y1="3.81" x2="16.51" y2="2.54" width="0.8128" layer="1"/>
 <wire x1="41.91" y1="10.16" x2="41.91" y2="17.78" width="0.8128" layer="1"/>
@@
 <wire x1="8.9154" y1="19.5834" x2="10.795" y2="19.5834" width="0.6096" layer="1"/>
 <wire x1="8.89" y1="19.558" x2="7.046" y2="19.558" width="0.8128" layer="1"/>
-<wire x1="7.046" y1="19.558" x2="6.858" y2="19.37" width="0.8128" layer="1"/>
+<wire x1="7.046" y1="19.558" x2="6.858" y2="19.42" width="0.8128" layer="1"/>
 </signal>
 <signal name="N$2">
@@
 <contactref element="C3" pad="2"/>
 <wire x1="16.002" y1="9.906" x2="15.24" y2="9.144" width="0.4064" layer="1"/>
-<wire x1="15.24" y1="9.144" x2="15.24" y2="6.665" width="0.4064" layer="1"/>
+<wire x1="15.24" y1="9.144" x2="15.24" y2="6.615" width="0.4064" layer="1"/>
 <wire x1="9.906" y1="9.906" x2="16.002" y2="9.906" width="0.4064" layer="16"/>
 <wire x1="9.906" y1="9.906" x2="12.065" y2="12.065" width="0.4064" layer="1"/>
@@
 <wire x1="17.145" y1="10.795" x2="17.145" y2="13.4366" width="0.4064" layer="1"/>
 <wire x1="19.05" y1="8.89" x2="17.145" y2="10.795" width="0.4064" layer="1"/>
-<wire x1="19.05" y1="6.665" x2="19.05" y2="8.89" width="0.4064" layer="1"/>
+<wire x1="19.05" y1="6.615" x2="19.05" y2="8.89" width="0.4064" layer="1"/>
 </signal>
 <signal name="N$4">
@@
 <wire x1="9.525" y1="8.255" x2="13.335" y2="12.065" width="0.4064" layer="1"/>
 <wire x1="13.335" y1="12.065" x2="13.335" y2="13.4366" width="0.4064" layer="1"/>
-<wire x1="8.575" y1="4.765" x2="7.62" y2="4.765" width="0.4064" layer="1"/>
+<wire x1="8.575" y1="4.765" x2="7.62" y2="4.815" width="0.4064" layer="1"/>
 </signal>
 <signal name="N$5">
 <contactref element="C1" pad="2"/>
 <contactref element="IC1" pad="1"/>
-<wire x1="7.62" y1="6.665" x2="7.62" y2="8.89" width="0.4064" layer="1"/>
+<wire x1="7.62" y1="6.615" x2="7.62" y2="8.89" width="0.4064" layer="1"/>
 <wire x1="10.795" y1="12.065" x2="10.795" y2="13.4366" width="0.4064" layer="1"/>
 <wire x1="7.62" y1="8.89" x2="10.795" y2="12.065" width="0.4064" layer="1"/>
@@
 <wire x1="13.208" y1="8.763" x2="15.875" y2="11.43" width="0.4064" layer="1"/>
 <wire x1="15.875" y1="11.43" x2="15.875" y2="13.4366" width="0.4064" layer="1"/>
-<wire x1="11.75" y1="4.765" x2="11.43" y2="4.765" width="0.4064" layer="1"/>
+<wire x1="11.75" y1="4.765" x2="11.43" y2="4.815" width="0.4064" layer="1"/>
 </signal>
 <signal name="N$7">
 <contactref element="C2" pad="2"/>
 <contactref element="IC1" pad="4"/>
-<wire x1="11.43" y1="6.665" x2="11.43" y2="8.89" width="0.4064" layer="1"/>
+<wire x1="11.43" y1="6.615" x2="11.43" y2="8.89" width="0.4064" layer="1"/>
 <wire x1="11.43" y1="8.89" x2="14.605" y2="12.065" width="0.4064" layer="1"/>
 <wire x1="14.605" y1="12.065" x2="14.605" y2="13.4366" width="0.4064" layer="1"/>
