File: projects/jphy.v1.3/jphy_v1.3.sch (EAGLE design)
At the start: 11 parts, among them IC1 MAX3232ESE, J1 RJ45-8X

Commit message: JPHY ver 1.3 (300 pcs)
Parts:
- C1, C2, C3, C4, C5: device rcl:C-EUC0805 -> ipc-7351-capacitor:CAPACITOR_0805
- R1: device rcl:R-EU_R0805 -> ipc-7351-resistor:RESISTOR_0805
Other:
- moved on the sheet: C1, C2, C3, C4, C5
Changed lines of the file:
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@@
 <?xml version="1.0" encoding="utf-8"?>
 <!DOCTYPE eagle SYSTEM "eagle.dtd">
-<eagle version="6.3">
+<eagle version="6.5.0">
 <drawing>
 <settings>
@@
 <setting verticaltext="up"/>
 </settings>
-<grid distance="0.1" unitdist="inch" unit="inch" style="lines" multiple="1" display="no" altdistance="0.01" altunitdist="inch" altunit="inch"/>
+<grid distance="0.1" unitdist="inch" unit="inch" style="lines" multiple="1" display="yes" altdistance="0.01" altunitdist="inch" altunit="inch"/>
 <layers>
 <layer number="1" name="Top" color="4" fill="1" visible="no" active="no"/>
@@
 <layer number="48" name="Document" color="7" fill="1" visible="no" active="no"/>
 <layer number="49" name="Reference" color="7" fill="1" visible="no" active="no"/>
+<layer number="50" name="dxf" color="7" fill="1" visible="no" active="no"/>
 <layer number="51" name="tDocu" color="7" fill="1" visible="no" active="no"/>
 <layer number="52" name="bDocu" color="7" fill="1" visible="no" active="no"/>
@@
 <layer number="97" name="Info" color="7" fill="1" visible="yes" active="yes"/>
 <layer number="98" name="Guide" color="6" fill="1" visible="yes" active="yes"/>
+<layer number="250" name="Descript" color="3" fill="1" visible="no" active="no"/>
+<layer number="251" name="SMDround" color="12" fill="11" visible="no" active="no"/>
 </layers>
 <schematic xreflabel="%F%N/%S.%C%R" xrefpart="/%S.%C%R">
@@
 <part name="FRAME1" library="frames" deviceset="DINA4_L" device="" value="Where is this value"/>
 <part name="IC1" library="maxim" deviceset="MAX3232*" device="SE" technology="E"/>
-<part name="C1" library="rcl" deviceset="C-EU" device="C0805" value="0.47 uF"/>
-<part name="C2" library="rcl" deviceset="C-EU" device="C0805" value="0.47 uF"/>
-<part name="C3" library="rcl" deviceset="C-EU" device="C0805" value="0.47 uF"/>
-<part name="C4" library="rcl" deviceset="C-EU" device="C0805" value="0.47 uF"/>
-<part name="C5" library="rcl" deviceset="C-EU" device="C0805" value="0.47 uF"/>
-<part name="R1" library="rcl" deviceset="R-EU_" device="R0805" value="270 R"/>
+<part name="C1" library="ipc-7351-capacitor" deviceset="CAPACITOR_" device="0805" value="0.47 uF"/>
+<part name="C2" library="ipc-7351-capacitor" deviceset="CAPACITOR_" device="0805" value="0.47 uF"/>
+<part name="C3" library="ipc-7351-capacitor" deviceset="CAPACITOR_" device="0805" value="0.47 uF"/>
+<part name="C4" library="ipc-7351-capacitor" deviceset="CAPACITOR_" device="0805" value="0.47 uF"/>
+<part name="C5" library="ipc-7351-capacitor" deviceset="CAPACITOR_" device="0805" value="0.47 uF"/>
+<part name="R1" library="ipc-7351-resistor" deviceset="RESISTOR_" device="0805" value="270 R"/>
 <part name="LED1" library="jlab" deviceset="LED" device="CHIP-LED0805" value="Green"/>
 <part name="J1" library="jlab" deviceset="RJ45" device="" technology="-8X"/>
@@
 <instance part="IC1" gate="G$1" x="142.24" y="116.84"/>
 <instance part="IC1" gate="P" x="73.66" y="53.34"/>
-<instance part="C1" gate="G$1" x="104.14" y="127" rot="R180"/>
-<instance part="C2" gate="G$1" x="78.74" y="127" rot="R180"/>
-<instance part="C3" gate="G$1" x="170.18" y="144.78"/>
-<instance part="C4" gate="G$1" x="200.66" y="124.46" rot="R180"/>
-<instance part="C5" gate="G$1" x="50.8" y="55.88"/>
+<instance part="C1" gate="G$1" x="104.14" y="129.54" rot="R90"/>
+<instance part="C2" gate="G$1" x="78.74" y="129.54" rot="R90"/>
+<instance part="C3" gate="G$1" x="170.18" y="142.24" rot="R270"/>
+<instance part="C4" gate="G$1" x="200.66" y="127" rot="R90"/>
+<instance part="C5" gate="G$1" x="50.8" y="55.88" rot="R270"/>
 <instance part="R1" gate="G$1" x="30.48" y="50.8" rot="R90"/>
 <instance part="LED1" gate="G$1" x="30.48" y="60.96"/>
@@
 </segment>
 <segment>
-<wire x1="50.8" y1="63.5" x2="50.8" y2="58.42" width="0.1524" layer="91"/>
+<wire x1="50.8" y1="63.5" x2="50.8" y2="60.96" width="0.1524" layer="91"/>
 <pinref part="C5" gate="G$1" pin="1"/>
 <pinref part="+3V1" gate="VCC" pin="VCC"/>
@@
 <segment>
 <wire x1="157.48" y1="127" x2="170.18" y2="127" width="0.1524" layer="91"/>
-<wire x1="170.18" y1="127" x2="170.18" y2="139.7" width="0.1524" layer="91"/>
+<wire x1="170.18" y1="127" x2="170.18" y2="137.16" width="0.1524" layer="91"/>
 <pinref part="IC1" gate="G$1" pin="V+"/>
 <pinref part="C3" gate="G$1" pin="2"/>
@@
 <wire x1="175.26" y1="121.92" x2="175.26" y2="134.62" width="0.1524" layer="91"/>
 <wire x1="175.26" y1="134.62" x2="200.66" y2="134.62" width="0.1524" layer="91"/>
-<wire x1="200.66" y1="134.62" x2="200.66" y2="129.54" width="0.1524" layer="91"/>
+<wire x1="200.66" y1="134.62" x2="200.66" y2="132.08" width="0.1524" layer="91"/>
 <pinref part="IC1" gate="G$1" pin="V-"/>
 <pinref part="C4" gate="G$1" pin="2"/>
@@
 <net name="N$5" class="0">
 <segment>
-<wire x1="104.14" y1="132.08" x2="104.14" y2="137.16" width="0.1524" layer="91"/>
+<wire x1="104.14" y1="134.62" x2="104.14" y2="137.16" width="0.1524" layer="91"/>
 <wire x1="104.14" y1="137.16" x2="114.3" y2="137.16" width="0.1524" layer="91"/>
 <wire x1="114.3" y1="137.16" x2="114.3" y2="129.54" width="0.1524" layer="91"/>
@@
 <net name="N$7" class="0">
 <segment>
-<wire x1="78.74" y1="132.08" x2="78.74" y2="137.16" width="0.1524" layer="91"/>
+<wire x1="78.74" y1="134.62" x2="78.74" y2="137.16" width="0.1524" layer="91"/>
 <wire x1="78.74" y1="137.16" x2="91.44" y2="137.16" width="0.1524" layer="91"/>
 <wire x1="91.44" y1="137.16" x2="91.44" y2="119.38" width="0.1524" layer="91"/>
