File: projects/boiler_themp/room_ind/room_ind.brd (EAGLE design)
At the start: 50 x 50 mm, 56 parts, among them Q5 TLV1117, U1 G2XX3---PW20, U2 TPS71533_DCK_5

Commit message: boiler room indicator - allign leds brightness
Parts:
- R10, R17, R18, R24, R25, R3, R30, R31, R4, R9: value 470 -> 1K
- R34: value 470 -> 4.7K
- R35: value 1K -> 10K
Changed lines of the file:
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@@
 <?xml version="1.0" encoding="utf-8"?>
 <!DOCTYPE eagle SYSTEM "eagle.dtd">
-<eagle version="6.3">
+<eagle version="6.5.0">
 <drawing>
 <settings>
@@
 <attribute name="VALUE" x="6.9088" y="34.544" size="1.27" layer="27" ratio="10" rot="R90"/>
 </element>
-<element name="R3" library="rcl" package="R0805" value="470" x="8.89" y="36.83" smashed="yes" rot="R90">
+<element name="R3" library="rcl" package="R0805" value="1K" x="8.89" y="36.83" smashed="yes" rot="R90">
 <attribute name="NAME" x="8.89" y="28.575" size="1.27" layer="25" rot="R90"/>
 <attribute name="VALUE" x="11.43" y="36.195" size="1.27" layer="27" rot="R90"/>
 </element>
-<element name="R4" library="rcl" package="0207/7" value="470" x="8.89" y="36.83" smashed="yes" rot="R90">
+<element name="R4" library="rcl" package="0207/7" value="1K" x="8.89" y="36.83" smashed="yes" rot="R90">
 <attribute name="VALUE" x="9.4488" y="34.544" size="1.27" layer="27" ratio="10" rot="R90"/>
 </element>
@@
 <attribute name="VALUE" x="14.5288" y="34.544" size="1.27" layer="27" ratio="10" rot="R90"/>
 </element>
-<element name="R9" library="rcl" package="R0805" value="470" x="16.51" y="36.83" smashed="yes" rot="R90">
+<element name="R9" library="rcl" package="R0805" value="1K" x="16.51" y="36.83" smashed="yes" rot="R90">
 <attribute name="NAME" x="16.51" y="28.575" size="1.27" layer="25" rot="R90"/>
 <attribute name="VALUE" x="19.05" y="36.195" size="1.27" layer="27" rot="R90"/>
 </element>
-<element name="R10" library="rcl" package="0207/7" value="470" x="16.51" y="36.83" smashed="yes" rot="R90">
+<element name="R10" library="rcl" package="0207/7" value="1K" x="16.51" y="36.83" smashed="yes" rot="R90">
 <attribute name="VALUE" x="17.0688" y="34.544" size="1.27" layer="27" ratio="10" rot="R90"/>
 </element>
@@
 <attribute name="VALUE" x="22.1488" y="34.544" size="1.27" layer="27" ratio="10" rot="R90"/>
 </element>
-<element name="R17" library="rcl" package="R0805" value="470" x="24.13" y="36.83" smashed="yes" rot="R90">
+<element name="R17" library="rcl" package="R0805" value="1K" x="24.13" y="36.83" smashed="yes" rot="R90">
 <attribute name="NAME" x="24.13" y="28.575" size="1.27" layer="25" rot="R90"/>
 <attribute name="VALUE" x="26.67" y="36.195" size="1.27" layer="27" rot="R90"/>
 </element>
-<element name="R18" library="rcl" package="0207/7" value="470" x="24.13" y="36.83" smashed="yes" rot="R90">
+<element name="R18" library="rcl" package="0207/7" value="1K" x="24.13" y="36.83" smashed="yes" rot="R90">
 <attribute name="VALUE" x="24.6888" y="34.544" size="1.27" layer="27" ratio="10" rot="R90"/>
 </element>
@@
 <attribute name="VALUE" x="29.7688" y="34.544" size="1.27" layer="27" ratio="10" rot="R90"/>
 </element>
-<element name="R24" library="rcl" package="R0805" value="470" x="31.75" y="36.83" smashed="yes" rot="R90">
+<element name="R24" library="rcl" package="R0805" value="1K" x="31.75" y="36.83" smashed="yes" rot="R90">
 <attribute name="VALUE" x="34.29" y="36.195" size="1.27" layer="27" rot="R90"/>
 </element>
-<element name="R25" library="rcl" package="0207/7" value="470" x="31.75" y="36.83" smashed="yes" rot="R90">
+<element name="R25" library="rcl" package="0207/7" value="1K" x="31.75" y="36.83" smashed="yes" rot="R90">
 <attribute name="NAME" x="31.623" y="28.575" size="1.27" layer="25" ratio="10" rot="R90"/>
 <attribute name="VALUE" x="32.3088" y="34.544" size="1.27" layer="27" ratio="10" rot="R90"/>
@@
 <attribute name="VALUE" x="37.3888" y="34.544" size="1.27" layer="27" ratio="10" rot="R90"/>
 </element>
-<element name="R30" library="rcl" package="R0805" value="470" x="39.37" y="36.83" smashed="yes" rot="R90">
+<element name="R30" library="rcl" package="R0805" value="1K" x="39.37" y="36.83" smashed="yes" rot="R90">
 <attribute name="VALUE" x="41.91" y="36.195" size="1.27" layer="27" rot="R90"/>
 </element>
-<element name="R31" library="rcl" package="0207/7" value="470" x="39.37" y="36.83" smashed="yes" rot="R90">
+<element name="R31" library="rcl" package="0207/7" value="1K" x="39.37" y="36.83" smashed="yes" rot="R90">
 <attribute name="NAME" x="39.243" y="28.575" size="1.27" layer="25" ratio="10" rot="R90"/>
 <attribute name="VALUE" x="39.9288" y="34.544" size="1.27" layer="27" ratio="10" rot="R90"/>
@@
 <attribute name="VALUE" x="46.99" y="5.715" size="1.27" layer="27"/>
 </element>
-<element name="R34" library="rcl" package="R0805" value="470" x="39.37" y="8.89" rot="R270"/>
-<element name="R35" library="rcl" package="R0805" value="1K" x="39.37" y="13.97" rot="R270"/>
+<element name="R34" library="rcl" package="R0805" value="4.7K" x="39.37" y="8.89" rot="R270"/>
+<element name="R35" library="rcl" package="R0805" value="10K" x="39.37" y="13.97" rot="R270"/>
 <element name="C1" library="rcl" package="C0805" value="0.47uF" x="7.62" y="46.99" rot="R270"/>
 <element name="C2" library="rcl" package="C0805" value="0.47uF" x="41.91" y="46.99" rot="R270"/>
