File: projects/boiler_themp/room_ind/room_ind.sch (EAGLE design)
At the start: 56 parts, among them Q5 TLV1117, U1 G2XX3---PW20, U2 TPS71533_DCK_5

Commit message: boiler room indicator - allign leds brightness
Parts:
- R10, R17, R18, R24, R25, R3, R30, R31, R4, R9: value 470 -> 1K
- R34: value 470 -> 4.7K
- R35: value 1K -> 10K
Changed lines of the file:
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@@
 <?xml version="1.0" encoding="utf-8"?>
 <!DOCTYPE eagle SYSTEM "eagle.dtd">
-<eagle version="6.3">
+<eagle version="6.5.0">
 <drawing>
 <settings>
@@
 <part name="R1" library="rcl" deviceset="R-EU_" device="R0805" value="470"/>
 <part name="R2" library="rcl" deviceset="R-EU_" device="0207/7" value="470"/>
-<part name="R3" library="rcl" deviceset="R-EU_" device="R0805" value="470"/>
-<part name="R4" library="rcl" deviceset="R-EU_" device="0207/7" value="470"/>
+<part name="R3" library="rcl" deviceset="R-EU_" device="R0805" value="1K"/>
+<part name="R4" library="rcl" deviceset="R-EU_" device="0207/7" value="1K"/>
 <part name="R5" library="rcl" deviceset="R-EU_" device="R0805" value="470"/>
 <part name="R6" library="rcl" deviceset="R-EU_" device="0207/7" value="470"/>
@@
 <part name="R7" library="rcl" deviceset="R-EU_" device="R0805" value="470"/>
 <part name="R8" library="rcl" deviceset="R-EU_" device="0207/7" value="470"/>
-<part name="R9" library="rcl" deviceset="R-EU_" device="R0805" value="470"/>
-<part name="R10" library="rcl" deviceset="R-EU_" device="0207/7" value="470"/>
+<part name="R9" library="rcl" deviceset="R-EU_" device="R0805" value="1K"/>
+<part name="R10" library="rcl" deviceset="R-EU_" device="0207/7" value="1K"/>
 <part name="R11" library="rcl" deviceset="R-EU_" device="R0805" value="470"/>
 <part name="R12" library="rcl" deviceset="R-EU_" device="0207/7" value="470"/>
@@
 <part name="R13" library="rcl" deviceset="R-EU_" device="R0805" value="470"/>
 <part name="R14" library="rcl" deviceset="R-EU_" device="0207/7" value="470"/>
-<part name="R17" library="rcl" deviceset="R-EU_" device="R0805" value="470"/>
-<part name="R18" library="rcl" deviceset="R-EU_" device="0207/7" value="470"/>
+<part name="R17" library="rcl" deviceset="R-EU_" device="R0805" value="1K"/>
+<part name="R18" library="rcl" deviceset="R-EU_" device="0207/7" value="1K"/>
 <part name="R19" library="rcl" deviceset="R-EU_" device="R0805" value="470"/>
 <part name="R20" library="rcl" deviceset="R-EU_" device="0207/7" value="470"/>
@@
 <part name="R21" library="rcl" deviceset="R-EU_" device="R0805" value="470"/>
 <part name="R23" library="rcl" deviceset="R-EU_" device="0207/7" value="470"/>
-<part name="R24" library="rcl" deviceset="R-EU_" device="R0805" value="470"/>
-<part name="R25" library="rcl" deviceset="R-EU_" device="0207/7" value="470"/>
+<part name="R24" library="rcl" deviceset="R-EU_" device="R0805" value="1K"/>
+<part name="R25" library="rcl" deviceset="R-EU_" device="0207/7" value="1K"/>
 <part name="R26" library="rcl" deviceset="R-EU_" device="R0805" value="470"/>
 <part name="R27" library="rcl" deviceset="R-EU_" device="0207/7" value="470"/>
@@
 <part name="R28" library="rcl" deviceset="R-EU_" device="R0805" value="470"/>
 <part name="R29" library="rcl" deviceset="R-EU_" device="0207/7" value="470"/>
-<part name="R30" library="rcl" deviceset="R-EU_" device="R0805" value="470"/>
-<part name="R31" library="rcl" deviceset="R-EU_" device="0207/7" value="470"/>
+<part name="R30" library="rcl" deviceset="R-EU_" device="R0805" value="1K"/>
+<part name="R31" library="rcl" deviceset="R-EU_" device="0207/7" value="1K"/>
 <part name="R32" library="rcl" deviceset="R-EU_" device="R0805" value="470"/>
 <part name="R33" library="rcl" deviceset="R-EU_" device="0207/7" value="470"/>
 <part name="P+11" library="supply1" deviceset="+3V3" device=""/>
 <part name="JP2" library="SparkFun-Connectors" deviceset="M01" device="PTH" value="RXD_5V"/>
-<part name="R34" library="rcl" deviceset="R-EU_" device="R0805" value="470"/>
-<part name="R35" library="rcl" deviceset="R-EU_" device="R0805" value="1K"/>
+<part name="R34" library="rcl" deviceset="R-EU_" device="R0805" value="4.7K"/>
+<part name="R35" library="rcl" deviceset="R-EU_" device="R0805" value="10K"/>
 <part name="GND1" library="supply1" deviceset="GND" device=""/>
 <part name="C1" library="rcl" deviceset="C-EU" device="C0805" value="0.47uF"/>
