File: projects/boiler_themp/upper_measure/upper_meter.brd (EAGLE design)
At the start: 50 x 50 mm, 48 parts, among them Q5 TLV1117, T2 MBT3906, U1 G2XX3---PW20, U2 TPS71533_DCK_5

Commit message: save unfinished changes in boiler schematics
Parts:
- removed JP11: P13, SparkFun:1X01
- removed JP8: P10, SparkFun:1X01
- added C12: 100 uF, rcl:E2,5-7
- added OK2: MOC3023M, optocoupler:DIL06
- added R17, R18: 4.7K, rcl:R0805
- R21: value 470 -> 1K
Connections:
- new net N$10: C12.+, R17.1
- new net N$11: OK2.2, R18.1
- net +3V3: now also OK2.1
- net GND: now also C12.-
- net P10: now also R17.2; no longer JP8.1
- net P13: now also R18.2; no longer JP11.1
Routing:
- net P13: track 15.9 -> 1.98 mm
- net P10: track 8.69 -> 8.14 mm
Changed lines of the file:
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@@
 <?xml version="1.0" encoding="utf-8"?>
 <!DOCTYPE eagle SYSTEM "eagle.dtd">
-<eagle version="6.3">
+<eagle version="6.5.0">
 <drawing>
 <settings>
@@
 <attribute name="VALUE" x="26.67" y="1.27" size="1.27" layer="27" rot="R90"/>
 </element>
-<element name="R21" library="rcl" package="R0805" value="470" x="24.13" y="6.35" smashed="yes" rot="R270">
+<element name="R21" library="rcl" package="R0805" value="1K" x="24.13" y="6.35" smashed="yes" rot="R270">
 <attribute name="NAME" x="30.48" y="12.065" size="1.27" layer="25" rot="R270"/>
 <attribute name="VALUE" x="21.59" y="6.985" size="1.27" layer="27" rot="R270"/>
@@
 <attribute name="VALUE" x="35.56" y="1.905" size="1.27" layer="27"/>
 </element>
-<element name="JP8" library="SparkFun" package="1X01" value="P10" x="39.37" y="5.08" smashed="yes">
-<attribute name="NAME" x="39.4462" y="7.5438" size="0.8128" layer="25" rot="R90"/>
-<attribute name="VALUE" x="38.1" y="1.905" size="1.27" layer="27"/>
-</element>
 <element name="JP9" library="SparkFun" package="1X01" value="P11" x="48.26" y="12.7" smashed="yes" rot="R270">
 <attribute name="NAME" x="43.7388" y="12.6238" size="0.8128" layer="25"/>
@@
 <attribute name="VALUE" x="45.085" y="11.43" size="1.27" layer="27" rot="R270"/>
 </element>
-<element name="JP11" library="SparkFun" package="1X01" value="P13" x="48.26" y="7.62" smashed="yes" rot="R270">
-<attribute name="NAME" x="43.7388" y="7.5438" size="0.8128" layer="25"/>
-<attribute name="VALUE" x="45.085" y="8.89" size="1.27" layer="27" rot="R270"/>
-</element>
 <element name="LED2" library="jlab" package="CHIP-LED0805" value="GREEN" x="21.59" y="2.54" smashed="yes">
 <attribute name="NAME" x="29.845" y="3.81" size="1.27" layer="25" rot="R90"/>
@@
 <attribute name="NAME" x="26.67" y="12.065" size="1.27" layer="25" rot="R270"/>
 <attribute name="VALUE" x="16.51" y="6.985" size="1.27" layer="27" rot="R270"/>
+</element>
+<element name="R17" library="rcl" package="R0805" value="4.7K" x="2.54" y="-3.81"/>
+<element name="C12" library="rcl" package="E2,5-7" value="100 uF" x="3.81" y="-11.43"/>
+<element name="R18" library="rcl" package="R0805" value="4.7K" x="2.54" y="-19.05"/>
+<element name="OK2" library="optocoupler" package="DIL06" value="MOC3023M" x="-6.35" y="-13.97">
+<attribute name="OC_NEWARK" value="72K8896" x="-6.35" y="-13.97" size="1.778" layer="27" display="off"/>
+<attribute name="MPN" value="MOC3023-M" x="-6.35" y="-13.97" size="1.778" layer="27" display="off"/>
+<attribute name="MF" value="FAIRCHILD SEMICONDUCTOR" x="-6.35" y="-13.97" size="1.778" layer="27" display="off"/>
+<attribute name="OC_FARNELL" value="1021367" x="-6.35" y="-13.97" size="1.778" layer="27" display="off"/>
 </element>
 </elements>
@@
 <wire x1="26.67" y1="19.37" x2="26.67" y2="15.24" width="0.3048" layer="1"/>
 <wire x1="48.26" y1="41.91" x2="48.26" y2="31.75" width="0.6096" layer="1"/>
+<contactref element="C12" pad="-"/>
+<wire x1="48.26" y1="36.83" x2="48.26" y2="39.37" width="0" layer="19" extent="1-1"/>
+<wire x1="48.26" y1="34.29" x2="48.26" y2="36.83" width="0" layer="19" extent="1-1"/>
+<wire x1="48.26" y1="41.91" x2="48.26" y2="39.37" width="0" layer="19" extent="1-1"/>
+<wire x1="40.64" y1="36.515" x2="48.26" y2="36.83" width="0" layer="19" extent="1-1"/>
+<wire x1="38.735" y1="40.64" x2="39.055" y2="36.515" width="0" layer="19" extent="1-1"/>
+<wire x1="38.735" y1="45.085" x2="39.055" y2="40.96" width="0" layer="19" extent="1-1"/>
+<wire x1="39.055" y1="32.07" x2="38.735" y2="36.195" width="0" layer="19" extent="1-1"/>
+<wire x1="39.155" y1="27.725" x2="38.735" y2="31.75" width="0" layer="19" extent="1-1"/>
+<wire x1="33.9051" y1="19.41" x2="38.735" y2="27.305" width="0" layer="19" extent="1-1"/>
+<wire x1="17.145" y1="13.97" x2="16.27" y2="16.97" width="0" layer="19" extent="1-1"/>
+<wire x1="19.05" y1="9.525" x2="17.145" y2="13.97" width="0" layer="19" extent="1-1"/>
+<wire x1="21.59" y1="9.525" x2="19.05" y2="9.525" width="0" layer="19" extent="1-1"/>
+<wire x1="24.13" y1="9.525" x2="21.59" y2="9.525" width="0" layer="19" extent="1-1"/>
+<wire x1="8.89" y1="14.92" x2="15.0114" y2="13.97" width="0" layer="19" extent="1-1"/>
+<wire x1="8.89" y1="3.81" x2="19.05" y2="7.3" width="0" layer="19" extent="1-1"/>
+<wire x1="48.26" y1="17.78" x2="40.64" y2="27.725" width="0" layer="19" extent="1-1"/>
+<wire x1="24.13" y1="39.69" x2="38.735" y2="40.64" width="0" layer="19" extent="1-1"/>
+<wire x1="5.08" y1="-11.43" x2="8.89" y2="3.81" width="0" layer="19" extent="1-1"/>
+<wire x1="39.37" y1="2.54" x2="24.13" y2="7.3" width="0" layer="19" extent="1-1"/>
 </signal>
 <signal name="TXD">
@@
 <vertex x="0" y="1"/>
 </polygon>
+<contactref element="OK2" pad="1"/>
+<wire x1="20.32" y1="2.54" x2="-8.89" y2="-17.78" width="0" layer="19" extent="1-1"/>
 </signal>
 <signal name="N$9">
@@
 <signal name="P13">
 <contactref element="U1" pad="13"/>
-<contactref element="JP11" pad="1"/>
 <wire x1="38.455" y1="19.41" x2="38.455" y2="17.425" width="0.3048" layer="1"/>
-<wire x1="38.455" y1="17.425" x2="48.26" y2="7.62" width="0.3048" layer="1"/>
+<contactref element="R18" pad="2"/>
+<wire x1="3.49" y1="-19.05" x2="38.455" y2="17.425" width="0" layer="19" extent="1-1"/>
 </signal>
 <signal name="P12">
@@
 </signal>
 <signal name="P10">
-<contactref element="JP8" pad="1"/>
 <contactref element="U1" pad="10"/>
-<wire x1="39.37" y1="5.08" x2="39.7549" y2="5.4649" width="0.3048" layer="1"/>
 <wire x1="39.7549" y1="5.4649" x2="39.7549" y2="13.6099" width="0.3048" layer="1"/>
+<contactref element="R17" pad="2"/>
+<wire x1="3.49" y1="-3.81" x2="39.7549" y2="5.4649" width="0" layer="19" extent="1-1"/>
 </signal>
 <signal name="RXD">
@@
 <wire x1="7.62" y1="43.18" x2="8.89" y2="43.18" width="0.8128" layer="1"/>
 </signal>
+<signal name="N$10">
+<contactref element="C12" pad="+"/>
+<contactref element="R17" pad="1"/>
+<wire x1="1.59" y1="-3.81" x2="2.54" y2="-11.43" width="0" layer="19" extent="1-1"/>
+</signal>
+<signal name="N$11">
+<contactref element="R18" pad="1"/>
+<contactref element="OK2" pad="2"/>
+<wire x1="1.59" y1="-19.05" x2="-6.35" y2="-17.78" width="0" layer="19" extent="1-1"/>
+</signal>
 </signals>
