File: projects/boiler_themp/upper_measure/upper_meter.sch (EAGLE design)
At the start: 48 parts, among them Q5 TLV1117, T2 MBT3906, U1 G2XX3---PW20, U2 TPS71533_DCK_5

Commit message: save unfinished changes in boiler schematics
Parts:
- removed JP11: P13, SparkFun:M01PTH
- removed JP8: P10, SparkFun:M01PTH
- added C12: 100 uF, rcl:CPOL-EUE2.5-7
- added OK2: MOC3023M, optocoupler:MOC3023M
- added R17, R18: 4.7K, rcl:R-EU_R0805
- R21: value 470 -> 1K
Connections:
- new net N$10: C12.+, R17.1
- new net N$11: OK2.C, R18.1
- net +3V3: now also OK2.A
- net GND: now also C12.-
- net P10: now also R17.2; no longer JP8.1
- net P13: now also R18.2; no longer JP11.1
Other:
- note added: "RC"
- note added: "TRIAC"
Changed lines of the file:
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@@
 <?xml version="1.0" encoding="utf-8"?>
 <!DOCTYPE eagle SYSTEM "eagle.dtd">
-<eagle version="6.3">
+<eagle version="6.5.0">
 <drawing>
 <settings>
@@
 <layer number="91" name="Nets" color="2" fill="1" visible="yes" active="yes"/>
 <layer number="92" name="Busses" color="1" fill="1" visible="yes" active="yes"/>
-<layer number="93" name="Pins" color="2" fill="1" visible="yes" active="yes"/>
+<layer number="93" name="Pins" color="2" fill="1" visible="no" active="yes"/>
 <layer number="94" name="Symbols" color="4" fill="1" visible="yes" active="yes"/>
 <layer number="95" name="Names" color="7" fill="1" visible="yes" active="yes"/>
@@
 <layer number="98" name="Guide" color="6" fill="1" visible="yes" active="yes"/>
 <layer number="100" name="Muster" color="7" fill="1" visible="no" active="no"/>
-<layer number="101" name="Patch_Top" color="12" fill="4" visible="no" active="yes"/>
-<layer number="102" name="Vscore" color="7" fill="1" visible="no" active="yes"/>
-<layer number="103" name="tMap" color="7" fill="1" visible="no" active="yes"/>
-<layer number="104" name="Name" color="16" fill="1" visible="no" active="yes"/>
 <layer number="105" name="tPlate" color="7" fill="1" visible="no" active="yes"/>
 <layer number="106" name="bPlate" color="7" fill="1" visible="no" active="yes"/>
@@
 <layer number="144" name="Drill_legend" color="7" fill="1" visible="no" active="yes"/>
 <layer number="151" name="HeatSink" color="7" fill="1" visible="no" active="yes"/>
-<layer number="200" name="200bmp" color="1" fill="10" visible="no" active="yes"/>
-<layer number="201" name="201bmp" color="2" fill="10" visible="no" active="yes"/>
-<layer number="202" name="202bmp" color="3" fill="10" visible="no" active="yes"/>
-<layer number="203" name="203bmp" color="4" fill="10" visible="no" active="yes"/>
-<layer number="204" name="204bmp" color="5" fill="10" visible="no" active="yes"/>
-<layer number="205" name="205bmp" color="6" fill="10" visible="no" active="yes"/>
-<layer number="206" name="206bmp" color="7" fill="10" visible="no" active="yes"/>
-<layer number="207" name="207bmp" color="8" fill="10" visible="no" active="yes"/>
-<layer number="208" name="208bmp" color="9" fill="10" visible="no" active="yes"/>
-<layer number="209" name="209bmp" color="7" fill="1" visible="no" active="yes"/>
-<layer number="210" name="210bmp" color="7" fill="1" visible="no" active="yes"/>
-<layer number="211" name="211bmp" color="7" fill="1" visible="no" active="yes"/>
-<layer number="212" name="212bmp" color="7" fill="1" visible="no" active="yes"/>
-<layer number="213" name="213bmp" color="7" fill="1" visible="no" active="yes"/>
-<layer number="214" name="214bmp" color="7" fill="1" visible="no" active="yes"/>
-<layer number="215" name="215bmp" color="7" fill="1" visible="no" active="yes"/>
-<layer number="216" name="216bmp" color="7" fill="1" visible="no" active="yes"/>
 <layer number="217" name="217bmp" color="18" fill="1" visible="no" active="no"/>
 <layer number="218" name="218bmp" color="19" fill="1" visible="no" active="no"/>
@@
 <layer number="250" name="Descript" color="3" fill="1" visible="no" active="no"/>
 <layer number="251" name="SMDround" color="12" fill="11" visible="no" active="no"/>
-<layer number="254" name="cooling" color="7" fill="1" visible="no" active="yes"/>
 </layers>
 <schematic xreflabel="%F%N/%S.%C%R" xrefpart="/%S.%C%R">
@@
 <part name="GND5" library="supply1" deviceset="GND" device=""/>
 <part name="LED1" library="jlab" deviceset="LED" device="CHIP-LED0805" value="BLUE"/>
-<part name="R21" library="rcl" deviceset="R-EU_" device="R0805" value="470"/>
+<part name="R21" library="rcl" deviceset="R-EU_" device="R0805" value="1K"/>
 <part name="GND16" library="supply1" deviceset="GND" device=""/>
 <part name="C10" library="rcl" deviceset="C-EU" device="C0805" value="2.2nf"/>
@@
 <part name="JP6" library="SparkFun" deviceset="M01" device="PTH" value="P08"/>
 <part name="JP7" library="SparkFun" deviceset="M01" device="PTH" value="P09"/>
-<part name="JP8" library="SparkFun" deviceset="M01" device="PTH" value="P10"/>
 <part name="JP9" library="SparkFun" deviceset="M01" device="PTH" value="P11"/>
 <part name="JP10" library="SparkFun" deviceset="M01" device="PTH" value="P12"/>
-<part name="JP11" library="SparkFun" deviceset="M01" device="PTH" value="P13"/>
 <part name="LED2" library="jlab" deviceset="LED" device="CHIP-LED0805" value="GREEN"/>
 <part name="R15" library="rcl" deviceset="R-EU_" device="R0805" value="1K"/>
@@
 <part name="P+2" library="supply1" deviceset="+5V" device=""/>
 <part name="P+5" library="supply1" deviceset="+3V3" device=""/>
+<part name="R17" library="rcl" deviceset="R-EU_" device="R0805" value="4.7K"/>
+<part name="C12" library="rcl" deviceset="CPOL-EU" device="E2.5-7" value="100 uF"/>
+<part name="GND21" library="supply1" deviceset="GND" device=""/>
+<part name="P+6" library="supply1" deviceset="+3V3" device=""/>
+<part name="R18" library="rcl" deviceset="R-EU_" device="R0805" value="4.7K"/>
+<part name="OK2" library="optocoupler" deviceset="MOC30*M" device="" technology="23"/>
 </parts>
 <sheets>
@@
 <wire x1="378.46" y1="149.86" x2="355.6" y2="149.86" width="0.1524" layer="97"/>
 <text x="358.14" y="243.84" size="1.778" layer="97">Zero Cross Det</text>
+<text x="358.14" y="203.2" size="1.778" layer="97">RC</text>
+<text x="358.14" y="187.96" size="1.778" layer="97">TRIAC</text>
 </plain>
 <instances>
@@
 <attribute name="NAME" x="195.58" y="180.086" size="1.778" layer="95"/>
 </instance>
-<instance part="JP8" gate="G$1" x="190.5" y="177.8" smashed="yes" rot="R180">
-<attribute name="VALUE" x="195.58" y="177.8" size="1.778" layer="96"/>
-<attribute name="NAME" x="195.58" y="175.006" size="1.778" layer="95"/>
-</instance>
 <instance part="JP9" gate="G$1" x="190.5" y="172.72" smashed="yes" rot="R180">
 <attribute name="VALUE" x="195.58" y="172.72" size="1.778" layer="96"/>
@@
 <attribute name="VALUE" x="195.58" y="167.64" size="1.778" layer="96"/>
 <attribute name="NAME" x="195.58" y="164.846" size="1.778" layer="95"/>
-</instance>
-<instance part="JP11" gate="G$1" x="190.5" y="162.56" smashed="yes" rot="R180">
-<attribute name="VALUE" x="195.58" y="162.56" size="1.778" layer="96"/>
-<attribute name="NAME" x="195.58" y="159.766" size="1.778" layer="95"/>
 </instance>
 <instance part="LED2" gate="G$1" x="142.24" y="35.56" smashed="yes">
@@
 <attribute name="VALUE" x="144.78" y="43.18" size="1.778" layer="96"/>
 </instance>
+<instance part="R17" gate="G$1" x="195.58" y="127" smashed="yes" rot="R180">
+<attribute name="NAME" x="194.0814" y="130.81" size="1.778" layer="95" rot="R90"/>
+<attribute name="VALUE" x="196.85" y="130.81" size="1.778" layer="96" rot="R90"/>
+</instance>
+<instance part="C12" gate="G$1" x="203.2" y="119.38"/>
+<instance part="GND21" gate="1" x="203.2" y="104.14"/>
+<instance part="P+6" gate="G$1" x="203.2" y="81.28" smashed="yes">
+<attribute name="VALUE" x="205.74" y="81.28" size="1.778" layer="96"/>
+</instance>
+<instance part="R18" gate="G$1" x="198.12" y="66.04" smashed="yes" rot="R180">
+<attribute name="NAME" x="196.6214" y="69.85" size="1.778" layer="95" rot="R90"/>
+<attribute name="VALUE" x="199.39" y="69.85" size="1.778" layer="96" rot="R90"/>
+</instance>
+<instance part="OK2" gate="-1" x="220.98" y="71.12"/>
 </instances>
 <busses>
@@
 <wire x1="127" y1="17.78" x2="127" y2="15.24" width="0.1524" layer="91"/>
 </segment>
+<segment>
+<pinref part="GND21" gate="1" pin="GND"/>
+<pinref part="C12" gate="G$1" pin="-"/>
+<wire x1="203.2" y1="106.68" x2="203.2" y2="114.3" width="0.1524" layer="91"/>
+</segment>
 </net>
 <net name="RXD" class="0">
@@
 <junction x="111.76" y="60.96"/>
 </segment>
+<segment>
+<pinref part="OK2" gate="-1" pin="A"/>
+<pinref part="P+6" gate="G$1" pin="+3V3"/>
+<wire x1="210.82" y1="76.2" x2="203.2" y2="76.2" width="0.1524" layer="91"/>
+<wire x1="203.2" y1="76.2" x2="203.2" y2="78.74" width="0.1524" layer="91"/>
+</segment>
 </net>
 <net name="N$9" class="0">
@@
 <net name="P10" class="0">
 <segment>
-<pinref part="JP8" gate="G$1" pin="1"/>
-<wire x1="182.88" y1="177.8" x2="162.56" y2="177.8" width="0.1524" layer="91"/>
-<label x="165.1" y="177.8" size="1.778" layer="95"/>
-</segment>
-<segment>
 <pinref part="U1" gate="G$1" pin="10"/>
 <wire x1="81.28" y1="198.12" x2="100.33" y2="198.12" width="0.1524" layer="91"/>
 <label x="83.82" y="198.12" size="1.778" layer="95"/>
 </segment>
+<segment>
+<pinref part="R17" gate="G$1" pin="2"/>
+<wire x1="190.5" y1="127" x2="165.1" y2="127" width="0.1524" layer="91"/>
+<label x="166.37" y="127.762" size="1.778" layer="95"/>
+</segment>
 </net>
 <net name="P13" class="0">
@@
 </segment>
 <segment>
-<pinref part="JP11" gate="G$1" pin="1"/>
-<wire x1="182.88" y1="162.56" x2="162.56" y2="162.56" width="0.1524" layer="91"/>
-<label x="165.1" y="162.56" size="1.778" layer="95"/>
+<pinref part="R18" gate="G$1" pin="2"/>
+<wire x1="193.04" y1="66.04" x2="165.1" y2="66.04" width="0.1524" layer="91"/>
+<label x="167.386" y="66.802" size="1.778" layer="95"/>
 </segment>
 </net>
@@
 </segment>
 </net>
+<net name="N$10" class="0">
+<segment>
+<pinref part="C12" gate="G$1" pin="+"/>
+<pinref part="R17" gate="G$1" pin="1"/>
+<wire x1="203.2" y1="121.92" x2="203.2" y2="127" width="0.1524" layer="91"/>
+<wire x1="203.2" y1="127" x2="200.66" y2="127" width="0.1524" layer="91"/>
+</segment>
+</net>
+<net name="N$11" class="0">
+<segment>
+<pinref part="R18" gate="G$1" pin="1"/>
+<pinref part="OK2" gate="-1" pin="C"/>
+<wire x1="203.2" y1="66.04" x2="210.82" y2="66.04" width="0.1524" layer="91"/>
+</segment>
+</net>
